File: Receiver.sch (EAGLE design)
At the start: 28 parts, among them J1 SD_CARD_SOCKET, U1 PIC18F47Q84, U2 915MHz, U4 FT232RL, U5 DS1374C, U6 +12v, X1 BU-SMA-V, X2 PIC-PROG047

Commit message: Adding button inputs
Parts:
- added BTNA, BTNB: 53047-04, con-molex:53047-04
Connections:
- new net BTN1: BTNA-2.S, U1.RA2
- new net BTN2: BTNA-3.S, U1.RA1
- new net BTN3: BTNA-4.S, U1.RA0
- new net BTN4: BTNB-2.S, U1.RA5
- new net BTN5: BTNB-3.S, U1.RA4
- new net BTN6: BTNB-4.S, U1.RA3
- net GND: now also BTNA-1.S, BTNB-1.S
Changed lines of the file:
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@@
 <part name="I2C-DBG" library="SparkFun-Connectors" deviceset="CONN_03" device=""/>
 <part name="SUPPLY18" library="supply2" deviceset="GND" device=""/>
+<part name="BTNB" library="con-molex" deviceset="53?-04" device="047"/>
+<part name="BTNA" library="con-molex" deviceset="53?-04" device="047"/>
+<part name="SUPPLY19" library="supply2" deviceset="GND" device=""/>
 </parts>
 <sheets>
@@
 <instance part="I2C-DBG" gate="J$1" x="22.86" y="93.98"/>
 <instance part="SUPPLY18" gate="GND" x="30.48" y="88.9"/>
+<instance part="BTNB" gate="-1" x="-33.02" y="48.26"/>
+<instance part="BTNB" gate="-2" x="-7.62" y="60.96"/>
+<instance part="BTNB" gate="-3" x="-7.62" y="58.42"/>
+<instance part="BTNB" gate="-4" x="-7.62" y="55.88"/>
+<instance part="BTNA" gate="-1" x="-33.02" y="43.18"/>
+<instance part="BTNA" gate="-2" x="-7.62" y="40.64"/>
+<instance part="BTNA" gate="-3" x="-7.62" y="38.1"/>
+<instance part="BTNA" gate="-4" x="-7.62" y="35.56"/>
+<instance part="SUPPLY19" gate="GND" x="-35.56" y="40.64"/>
 </instances>
 <busses>
@@
 </segment>
 <segment>
-<pinref part="U6" gate="G$1" pin="GND"/>
 <pinref part="U6" gate="G$1" pin="GND"/>
 <pinref part="SUPPLY2" gate="GND" pin="GND"/>
@@
 <pinref part="SUPPLY18" gate="GND" pin="GND"/>
 </segment>
+<segment>
+<pinref part="BTNA" gate="-1" pin="S"/>
+<pinref part="SUPPLY19" gate="GND" pin="GND"/>
+<pinref part="BTNB" gate="-1" pin="S"/>
+<wire x1="-35.56" y1="48.26" x2="-35.56" y2="43.18" width="0.1524" layer="91"/>
+<junction x="-35.56" y="43.18"/>
+</segment>
 </net>
 <net name="SCK1" class="0">
@@
 </segment>
 </net>
+<net name="BTN1" class="0">
+<segment>
+<pinref part="BTNA" gate="-2" pin="S"/>
+<wire x1="-10.16" y1="40.64" x2="-15.24" y2="40.64" width="0.1524" layer="91"/>
+<label x="-15.24" y="40.64" size="1.778" layer="95" rot="R180"/>
+</segment>
+<segment>
+<pinref part="U1" gate="G$1" pin="RA2"/>
+<wire x1="35.56" y1="25.4" x2="30.48" y2="25.4" width="0.1524" layer="91"/>
+<label x="30.48" y="25.4" size="1.778" layer="95" rot="R180"/>
+</segment>
+</net>
+<net name="BTN2" class="0">
+<segment>
+<pinref part="BTNA" gate="-3" pin="S"/>
+<wire x1="-10.16" y1="38.1" x2="-15.24" y2="38.1" width="0.1524" layer="91"/>
+<label x="-15.24" y="38.1" size="1.778" layer="95" rot="R180"/>
+</segment>
+<segment>
+<pinref part="U1" gate="G$1" pin="RA1"/>
+<wire x1="35.56" y1="27.94" x2="30.48" y2="27.94" width="0.1524" layer="91"/>
+<label x="30.48" y="27.94" size="1.778" layer="95" rot="R180"/>
+</segment>
+</net>
+<net name="BTN3" class="0">
+<segment>
+<pinref part="BTNA" gate="-4" pin="S"/>
+<wire x1="-10.16" y1="35.56" x2="-15.24" y2="35.56" width="0.1524" layer="91"/>
+<label x="-15.24" y="35.56" size="1.778" layer="95" rot="R180"/>
+</segment>
+<segment>
+<pinref part="U1" gate="G$1" pin="RA0"/>
+<wire x1="35.56" y1="30.48" x2="30.48" y2="30.48" width="0.1524" layer="91"/>
+<label x="30.48" y="30.48" size="1.778" layer="95" rot="R180"/>
+</segment>
+</net>
+<net name="BTN6" class="0">
+<segment>
+<pinref part="BTNB" gate="-4" pin="S"/>
+<wire x1="-10.16" y1="55.88" x2="-12.7" y2="55.88" width="0.1524" layer="91"/>
+<label x="-12.7" y="55.88" size="1.778" layer="95" rot="R180"/>
+</segment>
+<segment>
+<pinref part="U1" gate="G$1" pin="RA3"/>
+<wire x1="35.56" y1="22.86" x2="30.48" y2="22.86" width="0.1524" layer="91"/>
+<label x="30.48" y="22.86" size="1.778" layer="95" rot="R180"/>
+</segment>
+</net>
+<net name="BTN5" class="0">
+<segment>
+<pinref part="BTNB" gate="-3" pin="S"/>
+<wire x1="-10.16" y1="58.42" x2="-12.7" y2="58.42" width="0.1524" layer="91"/>
+<label x="-12.7" y="58.42" size="1.778" layer="95" rot="R180"/>
+</segment>
+<segment>
+<pinref part="U1" gate="G$1" pin="RA4"/>
+<wire x1="35.56" y1="20.32" x2="30.48" y2="20.32" width="0.1524" layer="91"/>
+<label x="30.48" y="20.32" size="1.778" layer="95" rot="R180"/>
+</segment>
+</net>
+<net name="BTN4" class="0">
+<segment>
+<pinref part="BTNB" gate="-2" pin="S"/>
+<wire x1="-10.16" y1="60.96" x2="-12.7" y2="60.96" width="0.1524" layer="91"/>
+<label x="-12.7" y="60.96" size="1.778" layer="95" rot="R180"/>
+</segment>
+<segment>
+<pinref part="U1" gate="G$1" pin="RA5"/>
+<wire x1="35.56" y1="17.78" x2="30.48" y2="17.78" width="0.1524" layer="91"/>
+<label x="30.48" y="17.78" size="1.778" layer="95" rot="R180"/>
+</segment>
+</net>

Commit message: PCB updates
- Connected NC pins of DS1374 to GND
- Connected CLK_RST to PIC
- Moved I2C to default pins on PIC
Parts:
- C5: value (none) -> 10uF
- C6: value (none) -> 0.1uF
Connections:
- net RA8875-CS renamed RA8875_CS
- net RA8875-RST renamed RA8875_RST
- net RA8875-WAIT renamed RA8875_WAIT
- net SD-CS renamed SD_CS
- removed net N$9: U1.RC0
- removed net RA8875-INT: RA8875-10.S, RA8875-DBG.9, U1.RC4
- removed net RF-DIO0: SPI2-DBG.7, U1.RC7, U2.DIO0
- new net CLK_INT: U1.RB1, U5.!INT
- new net RA8875_INT: RA8875-10.S, RA8875-DBG.9, U1.RB0
- new net RF_DIO0: SPI2-DBG.7, U1.RB2, U2.DIO0
- new net SD_CD: J1.CD, U1.RC7
- net CLK_RST: now also U1.RA7/CLKIN
- net GND: now also U5.NC@1, U5.NC@2, U5.NC@3, U5.NC@4, U5.NC@5, U5.NC@6, U5.NC@7, U5.NC@8
- net MISO1: now also U1.RC1; no longer U1.RC2
- net MOSI1: now also U1.RC0; no longer U1.RC1
- net SCK1: now also U1.RC2; no longer U1.RC3
- net SCL: now also U1.RC3; no longer U1.RB5
- net SDA: now also U1.RC4; no longer U1.RB4
- net UARTRX: now also U1.RB4; no longer U1.RB2
- net UARTTX: now also U1.RB3; no longer U1.RB1
Other:
- moved on the sheet: TPSQW
